File: Air-Quality-PCB/Air-Quality-PCB.kicad_sch (KiCad schematic)
At the start: 35 parts, among them J1 Conn_01x03_Female, J10 Conn_01x02_Female, J11 Conn_01x10_Female, J12 Conn_01x02_Female, J13 Conn_01x10_Female, J14 Conn_01x03_Female, J15 Conn_01x03_Female, J16 Conn_01x04_Female, J17 Conn_01x04_Female, J18 Conn_01x05_Female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

Commit message: Add files via upload
Parts:
- added H1, H2, H3, H4: MountingHole, MountingHole:MountingHole_3.2mm_M3, symbol Mechanical:MountingHole
- added R10, R12, R13, R14, R15, R16, R3, R5, R9: 0, Resistor_SMD:R_1206_3216Metric, symbol Device:R_US
- J1: footprint (none) -> Connector_PinSocket_2.54mm:PinSocket_1x03_P2.54mm_Vertical
- J10, J12: footprint (none) -> Connector_PinHeader_2.54mm:PinHeader_1x02_P2.54mm_Vertical
- J11, J4: footprint (none) -> Connector_PinSocket_2.54mm:PinSocket_1x10_P2.54mm_Vertical
- J13, J2: footprint (none) -> Connector_PinHeader_2.54mm:PinHeader_1x10_P2.54mm_Vertical
- J14, J15, J21, J5, J6: footprint (none) -> Connector_PinHeader_2.54mm:PinHeader_1x03_P2.54mm_Vertical
- J16, J17, J20, J9: footprint (none) -> Connector_PinHeader_2.54mm:PinHeader_1x04_P2.54mm_Vertical
- J18, J19: footprint (none) -> Connector_PinSocket_2.54mm:PinSocket_1x05_P2.54mm_Vertical
- J3: footprint (none) -> Connector_PinHeader_2.54mm:PinHeader_1x08_P2.54mm_Vertical
- J7, J8: footprint (none) -> Connector_PinHeader_2.54mm:PinHeader_1x07_P2.54mm_Vertical
- R1, R2: value R_US -> 47k; footprint (none) -> Resistor_SMD:R_1206_3216Metric
- R11: renamed from 47k4; value R_US -> 47k; footprint (none) -> Resistor_SMD:R_1206_3216Metric
- R4: renamed from 47k1; value R_US -> 47k; footprint (none) -> Resistor_SMD:R_1206_3216Metric
- R6: renamed from 47k2; value R_US -> 47k; footprint (none) -> Resistor_SMD:R_1206_3216Metric
- R7: renamed from R3; value R_US -> 47k; footprint (none) -> Resistor_SMD:R_1206_3216Metric
- R8: renamed from 47k3; value R_US -> 47k; footprint (none) -> Resistor_SMD:R_1206_3216Metric
Connections:
- net +3.3V: now also R3.1, R5.1, R9.1
- net +5V: now also R10.1, R12.1; no longer J1.3 (Pin_3), J3.8 (Pin_8)
- net I2C_0 SCL: now also R15.1
- net I2C_0 SDA: now also R16.1
- net I2C_1 SCL: now also R13.1; no longer J17.3 (Pin_3)
- net I2C_1 SDA: now also R14.1; no longer J17.4 (Pin_4)
- net RX: now also J21.3 (Pin_3); no longer J21.2 (Pin_2)
- net TX: now also J21.2 (Pin_2); no longer J21.3 (Pin_3)
- net at J16.3 (Pin_3), J16.4 (Pin_4), Q1.3 (D): now also R3.2
- net at J18.2 (Pin_2), Q7.3 (D): now also R12.2
- net at J15.2 (Pin_2), J15.3 (Pin_3), J21.1 (Pin_1)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: now also R5.2
- net at J17.2 (Pin_2), Q5.3 (D): now also R9.2
- net at J19.3 (Pin_3), Q6.3 (D): now also R10.2
- new net: J17.3 (Pin_3), R13.2, R15.2
- new net: J17.4 (Pin_4), R14.2, R16.2
- new net 5V+: J1.3 (Pin_3), J3.8 (Pin_8)
Other:
- note added: "Battery connects to PowerBoost 500C, and is shared between both components"
- note added: "Circuit designed to be a HAT for the MSP430fr2355 Launchpad Microcontroller Pins bellow are modeled directly as if you were looking at a top down of the microcontroller Connectors J7-J8, J5-J6, J10-J12 will be shorted to there corosponsing pins with a jumper under normal operation (See data sheet)"
- note added: "P Channel mosfets for putting sensor to sleep N Channel mosfets for 3.3v to 5v level shifting 0 Ohm resistor to bypass sleep circuit if we opt for built in sensor sleep circuit"
- note added: "PowerBoost 500C Battery management/ Charging 5v boost circuit Battery input"
- note added: "TLV62569 3.3v stepdown circuit"
- company: (none) -> Portland State University Team 1
- title: (none) -> Air Quality PCB (2023)
- moved on the sheet: J3, J7, J8, Q2, Q5, R2, R7
